File: Dice.kicad_pcb (KiCad board)
At the start: 2 copper layers, 50.8 x 50.8 mm, 21 parts, among them IC1 CD74AC163, IC2 74AHC1G00, IC3 4511D, SW1 SW_DPDT_x2, SW2 SW_Push, U1 LM555N

Commit message: Dice revisited
Routing:
- net GND: track 244.2 -> 245.6 mm
- net BATT: track 32.8 -> 33.6 mm
Changed lines of the file:
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@@
     (links 60)
     (no_connects 0)
-    (area 26.340999 19.279799 77.291001 70.535802)
+    (area 13.082199 13.183799 64.032201 64.133801)
     (thickness 1.6)
     (drawings 4)
-    (tracks 332)
+    (tracks 333)
     (zones 0)
     (modules 21)
@@
   (segment (start 42.0624 48.26) (end 42.0624 47.76) (width 0.254) (layer F.Cu) (net 2))
   (segment (start 42.0624 47.76) (end 40.632 46.3296) (width 0.254) (layer F.Cu) (net 2))
+  (segment (start 49.3776 30.1244) (end 39.2684 30.1244) (width 0.381) (layer B.Cu) (net 3))
+  (via (at 39.2684 30.1244) (size 0.762) (drill 0.5842) (layers F.Cu B.Cu) (net 3))
+  (via (at 49.3776 30.1244) (size 0.762) (drill 0.5842) (layers F.Cu B.Cu) (net 3))
+  (segment (start 49.3776 31.3944) (end 49.3776 30.1244) (width 0.381) (layer F.Cu) (net 3))
   (segment (start 56.818082 36.752082) (end 58.3184 38.2524) (width 0.381) (layer F.Cu) (net 3))
   (segment (start 58.3184 38.2524) (end 58.3184 45.1104) (width 0.381) (layer F.Cu) (net 3))
@@
   (segment (start 39.5224 30.3784) (end 39.5224 31.1912) (width 0.381) (layer F.Cu) (net 3))
   (segment (start 39.5224 31.1912) (end 39.5224 33.02) (width 0.381) (layer F.Cu) (net 3))
-  (segment (start 49.3776 31.3944) (end 39.7256 31.3944) (width 0.381) (layer B.Cu) (net 3))
-  (segment (start 39.7256 31.3944) (end 39.5224 31.1912) (width 0.381) (layer B.Cu) (net 3))
-  (via (at 39.5224 31.1912) (size 0.762) (drill 0.5842) (layers F.Cu B.Cu) (net 3))
   (segment (start 50.1928 43.942) (end 54.067518 43.942) (width 0.381) (layer F.Cu) (net 3))
   (segment (start 49.3776 36.752082) (end 49.3776 31.3944) (width 0.381) (layer F.Cu) (net 3))
-  (via (at 49.3776 31.3944) (size 0.762) (drill 0.5842) (layers F.Cu B.Cu) (net 3))
   (segment (start 58.3184 45.1104) (end 57.8612 45.1104) (width 0.381) (layer F.Cu) (net 3))
   (segment (start 57.8612 45.1104) (end 56.6928 43.942) (width 0.381) (layer F.Cu) (net 3))
@@
   (segment (start 44.7548 17.018) (end 44.7548 16.114) (width 0.254) (layer F.Cu) (net 27))
   (segment (start 44.7548 16.114) (end 43.322 14.6812) (width 0.254) (layer F.Cu) (net 27))
-  (segment (start 50.6476 30.3784) (end 50.6476 32.1056) (width 0.381) (layer F.Cu) (net 29))
+  (segment (start 50.6476 29.0068) (end 50.6476 32.1056) (width 0.381) (layer F.Cu) (net 29))
   (segment (start 50.6476 32.1056) (end 53.1876 34.6456) (width 0.381) (layer F.Cu) (net 29))
-  (segment (start 36.1188 30.3784) (end 50.6476 30.3784) (width 0.381) (layer B.Cu) (net 29))
-  (via (at 50.6476 30.3784) (size 0.762) (drill 0.5842) (layers F.Cu B.Cu) (net 29))
+  (segment (start 34.9504 29.0068) (end 50.6476 29.0068) (width 0.381) (layer B.Cu) (net 29))
+  (via (at 50.6476 29.0068) (size 0.762) (drill 0.5842) (layers F.Cu B.Cu) (net 29))
+  (segment (start 33.6042 27.6606) (end 34.9504 29.0068) (width 0.381) (layer F.Cu) (net 29))
+  (via (at 34.9504 29.0068) (size 0.762) (drill 0.5842) (layers F.Cu B.Cu) (net 29))
+  (segment (start 33.401 27.6606) (end 33.6042 27.6606) (width 0.381) (layer F.Cu) (net 29))
   (segment (start 24.3078 27.6606) (end 33.401 27.6606) (width 0.381) (layer F.Cu) (net 29))
-  (segment (start 33.401 27.6606) (end 36.1188 30.3784) (width 0.381) (layer F.Cu) (net 29))
-  (via (at 36.1188 30.3784) (size 0.762) (drill 0.5842) (layers F.Cu B.Cu) (net 29))
 )
